Commit message: Modified camera position

File: Project4/my_robot/urdf/my_robot.xacro (robot description, xacro)
@@ -25,5 +25,5 @@
   </joint>
  <joint name="camera_optical_joint" type="fixed">
-    <origin xyz="0.2 0 0" rpy="0 0 0"/>
+    <origin xyz="0 0 0" rpy="-1.5707 0 -1.5707"/>
     <parent link="chassis"/>
     <child link="camera_link_optical"/>
